File: CurrentAmp.brd (EAGLE design)
At the start: 22.8 x 16.3 mm, 18 parts, among them J2 CONN_4SCREW_2.54

Commit message: Minor schematic cleanup
Parts:
- J2: value CONN_4SCREW_2.54 -> CONN_42.54_SCREW; device bschulz:1X04 -> bschulz:1X04_SCREW
- U1: value INA212 -> INA212DCK
- renumbered U$1 to U1, U$2 to U2
